File: kicad/genesis-3BP-remix.kicad_sch (KiCad schematic)
At the start: 89 parts, among them CON1 MD-90SM, J1 S, J10 XL, J11 CL, J12 YL, J2 R, J3 G, J4 B, J5 VS, J6 YR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

Commit message: Update cap pad change
Parts:
- C21, C22, C8: footprint Capacitor_Tantalum_SMD:CP_EIA-3528-21_Kemet-B -> Capacitor_Tantalum_SMD:CP_EIA-3528-15_AVX-H
Changed lines of the file:
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@@
       (effects (font (size 1.27 1.27)))
     )
-    (property "Footprint" "Capacitor_Tantalum_SMD:CP_EIA-3528-21_Kemet-B" (at 187.96 159.0548 0)
+    (property "Footprint" "Capacitor_Tantalum_SMD:CP_EIA-3528-15_AVX-H" (at 187.96 159.0548 0)
       (effects (font (size 1.27 1.27)) hide)
     )
@@
       (effects (font (size 1.27 1.27)))
     )
-    (property "Footprint" "Capacitor_Tantalum_SMD:CP_EIA-3528-21_Kemet-B" (at 185.42 46.0248 0)
+    (property "Footprint" "Capacitor_Tantalum_SMD:CP_EIA-3528-15_AVX-H" (at 185.42 46.0248 0)
       (effects (font (size 1.27 1.27)) hide)
     )
@@
       (effects (font (size 1.27 1.27)))
     )
-    (property "Footprint" "Capacitor_Tantalum_SMD:CP_EIA-3528-21_Kemet-B" (at 187.96 128.5748 0)
-      (effects (font (size 1.27 1.27)) hide)
-    )
+    (property "Footprint" "Capacitor_Tantalum_SMD:CP_EIA-3528-15_AVX-H" (at 187.96 128.5748 0)
+      (effects (font (size 1.27 1.27)) hide)
+    )

Commit message: Update silkscreen placement
Parts:
- U2: value TLV9062xD -> TL972IDR
Changed lines of the file:
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@@
       (effects (font (size 1.27 1.27)) (justify left))
     )
-    (property "Value" "TLV9062xD" (at 248.92 97.79 0)
+    (property "Value" "TL972IDR" (at 248.92 97.79 0)
       (effects (font (size 1.27 1.27)) (justify left))
     )
@@
       (effects (font (size 1.27 1.27)))
     )
-    (property "Value" "TLV9062xD" (at 154.94 121.92 0)
+    (property "Value" "TL972IDR" (at 154.94 121.92 0)
       (effects (font (size 1.27 1.27)))
     )
@@
       (effects (font (size 1.27 1.27)))
     )
-    (property "Value" "TLV9062xD" (at 154.94 156.21 0)
-      (effects (font (size 1.27 1.27)))
-    )
+    (property "Value" "TL972IDR" (at 154.94 156.21 0)
+      (effects (font (size 1.27 1.27)))
+    )
